File: Video Tutorial/kicad_tutorial/kicad_tutorial.kicad_pcb (KiCad board)
At the start: 4 copper layers, 50 parts, among them J1 Screw_Terminal_01x02, J2 SWD, J3 Conn_01x04, J4 Conn_01x04, J5 USB_B_Micro, Q1 AO3401A, SW1 SW_SPDT, U1 MP2359DJ-LF-Z, U2 STM32F405RGT6, U3 USBLC6-2SC6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

Commit message: Added notes for Chapter: Rough layout, finer details
Parts:
- moved D1 101.9 mm to (64.3, 153.0)
- moved C12 97.2 mm to (73.0, 135.5), turned to 180 degrees
- moved C11 95.3 mm to (73.0, 130.0)
- moved D3 92.7 mm to (100.7, 152.4)
- moved C10 92.0 mm to (65.5, 102.3)
- moved C4 92.0 mm to (59.8, 102.3)
- moved C5 92.0 mm to (59.8, 104.2)
- moved C6 92.0 mm to (59.8, 106.2)
- moved C7 92.0 mm to (62.7, 102.3)
- moved C8 92.0 mm to (62.7, 104.2)
- moved C9 92.0 mm to (62.7, 106.2)
- moved D2 90.5 mm to (116.0, 154.9)
- moved R3 89.9 mm to (63.2, 149.0)
- moved SW1 86.9 mm to (69.5, 117.3), turned to 180 degrees
- moved L2 86.2 mm to (116.3, 162.6)
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Connections:
- U1 pad 1: (no net) -> BUCK_BST
- U1 pad 2: (no net) -> GND
- U1 pad 3: (no net) -> BUCK_FB
- U1 pad 4: (no net) -> BUCK_EN
- U1 pad 5: (no net) -> BUCK_IN
- U1 pad 6: (no net) -> BUCK_SW

Commit message: Added notes for Chapter: Improving the layout, finer details
Parts:
- C10: value 1u -> 10n
- moved R9 67.5 mm to (61.3, 126.6)
- moved R10 65.1 mm to (63.5, 126.6)
- moved C16 47.2 mm to (79.8, 159.0), turned to 0 degrees
- moved C2 45.5 mm to (71.0, 147.1)
- moved R6 44.0 mm to (88.0, 152.8), turned to -90 degrees
- moved R7 43.5 mm to (89.8, 152.8), turned to 90 degrees
- moved C5 43.1 mm to (63.8, 147.1), turned to 180 degrees
- moved R8 42.3 mm to (91.5, 152.8), turned to -90 degrees
- moved C15 42.3 mm to (79.8, 155.8), turned to 0 degrees
- moved C6 41.1 mm to (72.3, 145.4)
- moved L2 39.9 mm to (78.2, 150.7), turned to -90 degrees
- moved C10 39.4 mm to (59.0, 141.2), turned to 90 degrees
- moved D2 38.7 mm to (78.4, 145.8)
- moved C1 38.4 mm to (74.8, 134.9), turned to 90 degrees
- moved J1 35.6 mm to (94.3, 146.2)
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Connections:
- C10 pad 1: +3.3V -> +3.3VA
- C9 pad 1: +3.3V -> +3.3VA
- F1 pad 1: +12V -> Net-(D3-K)
- F1 pad 2: Net-(Q1-D) -> Net-(F1-Pad2)
- FB1 pad 1: Net-(D3-K) -> Net-(F1-Pad2)
- L1 pad 2: +3.3V -> +3.3VA
- Q1 pad 3: Net-(Q1-D) -> +12V

Commit message: Added notes for Chapter: Tombstoning
Parts:
- moved H3 92.9 mm to (51.0, 159.0)
- moved H2 76.9 mm to (96.0, 159.0)
- moved H4 69.3 mm to (51.0, 119.0)
- moved H1 49.3 mm to (96.0, 119.0)
- moved R1 10.8 mm to (52.5, 130.2)
- moved D4 7.67 mm to (86.5, 116.8), turned to 180 degrees
- moved J2 7.19 mm to (78.0, 119.0)
- moved SW1 6.62 mm to (48.2, 129.5)
- moved C11 5.87 mm to (56.0, 140.5), turned to 180 degrees
- moved C12 5.63 mm to (56.0, 134.5), turned to 0 degrees
- moved R11 5.59 mm to (86.5, 119.0)
- moved J4 5.50 mm to (62.4, 158.6)
- moved J3 4.93 mm to (66.1, 119.5)
- moved U3 3.71 mm to (92.8, 129.8)
- moved J5 3.62 mm to (98.0, 129.5)
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Routing:
- net +3.3V: track 0.00 -> 11.5 mm
- net GND: track 0.00 -> 10.3 mm
- net HSE_IN: track 0.00 -> 8.68 mm
- net +3.3VA: track 0.00 -> 5.00 mm
- net Net-(C11-Pad1): track 0.00 -> 2.55 mm
- net Net-(U2-VCAP_2): track 0.00 -> 2.40 mm
- net Net-(U2-VCAP_1): track 0.00 -> 2.27 mm
- net LED_STATUS: track 0.00 -> 2.19 mm
- net Net-(D1-K): track 0.00 -> 2.02 mm
- net HSE_OUT: track 0.00 -> 1.74 mm
- added copper zone on In2.Cu, net +3.3V
- added copper zone on In1.Cu, net GND
Other:
- board outline added: 56 x 51 mm

Commit message: Added notes for Chapter: Design rules checker (DRC)
Parts:
- moved R9 5.42 mm to (65.5, 130.0)
- moved R10 3.41 mm to (63.0, 130.0), turned to 180 degrees
- moved C13 2.78 mm to (86.8, 146.2)
- moved U2 1.76 mm to (65.1, 139.2)
- moved C10 1.76 mm to (57.5, 141.2)
- moved C11 1.76 mm to (54.2, 140.5)
- moved C12 1.76 mm to (54.2, 134.5)
- moved C3 1.76 mm to (58.2, 131.9)
- moved C4 1.76 mm to (57.2, 135.0)
- moved C5 1.76 mm to (62.0, 147.0)
- moved C8 1.76 mm to (61.5, 131.6)
- moved C9 1.76 mm to (56.2, 141.2)
- moved D1 1.76 mm to (58.2, 145.5)
- moved L1 1.76 mm to (54.5, 142.9)
- moved R2 1.76 mm to (57.2, 138.2)
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Connections:
- J3 pad 2: I2C1_SDA -> I2C1_SCL
- J3 pad 3: I2C1_SCL -> I2C1_SDA
- J4 pad 2: UART3_RX -> UART3_TX
- J4 pad 3: UART3_TX -> UART3_RX
Routing:
- net GND: track 10.3 -> 70.5 mm, vias 0 -> 41
- net +3.3V: track 11.5 -> 68.3 mm, vias 0 -> 24
- net NRST: track 0.00 -> 27.2 mm, vias 0 -> 2
- net USB_D+: track 0.00 -> 24.5 mm
- net USB_D-: track 0.00 -> 23.7 mm
- net SWDIO: track 0.00 -> 21.6 mm
- net SW0: track 0.00 -> 18.5 mm
- net SWCLK: track 0.00 -> 17.0 mm
- net UART3_TX: track 0.00 -> 15.2 mm
- net UART3_RX: track 0.00 -> 14.8 mm
- net I2C1_SCL: track 0.00 -> 14.5 mm
- net I2C1_SDA: track 0.00 -> 14.3 mm
- net +5V: track 0.00 -> 14.0 mm
- net BOOT0: track 0.00 -> 13.1 mm
- net unconnected-(J5-Shield-Pad6): track 0.00 -> 12.6 mm
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
Commit message: Completed KiCad Tutorial Video
Parts:
- moved J1 84.5 mm to (169.1, 106.8)
- moved J4 84.5 mm to (137.1, 119.0)
- moved L2 84.5 mm to (153.0, 111.2)
- moved C1 84.5 mm to (147.8, 95.4)
- moved C10 84.5 mm to (132.2, 101.7)
- moved C11 84.5 mm to (129.0, 101.0)
- moved C12 84.5 mm to (129.0, 95.0)
- moved C13 84.5 mm to (161.5, 106.8)
- moved C14 84.5 mm to (157.0, 111.0)
- moved C15 84.5 mm to (154.5, 116.2)
- moved C16 84.5 mm to (154.5, 119.5)
- moved C2 84.5 mm to (144.5, 107.6)
- moved C3 84.5 mm to (133.0, 92.4)
- moved C4 84.5 mm to (132.0, 95.5)
- moved C5 84.5 mm to (136.8, 107.5)
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Other:
- board text added: "+"
- board text added: "3V3"
- board text added: "BOOT"
- board text added: "I2C"
- board text added: "POWER"
- board text added: "RUN"
- board text added: "STATUS"
- board text added: "STM32F4 TEST BOARD | REV 2"
- board text added: "SWD"
- board text added: "UART"
- board text added: "USB"
